File: linux/tutorials/modules/usb_display/schematic/usb_display/usb_display.kicad_pcb (KiCad board)
At the start: 2 copper layers, 100 x 99.9 mm, 105 parts, among them J1 Conn_01x04_Male, J10 Conn_01x03_Male, J11 Conn_02x01, J3 USB_C_Receptacle_USB2.0, J4 Conn_02x17_Odd_Even, J5 USB_C_Receptacle_USB2.0, J6 Conn_02x01, J7 Screw_Terminal_01x04, J8 Conn_01x03_Male, J9 Conn_02x01, Q1 BD250, Q2 Q_NMOS_GDS, Q3 Q_NMOS_GDS, Q4 Q_NMOS_GDS, Q5 Q_NMOS_GDS, Q6 Q_NMOS_GDS, Q7 Q_NMOS_GDS, Q8 Q_NMOS_GDS, Q9 Q_NMOS_GDS, SW1 B_0, SW10 B_9, SW11 B_10, SW12 B_11, SW13 B_12, SW14 B_13, SW15 B_14, SW16 B_15, SW17 SW_Push_Rst, SW18 B_ENTER, SW2 B_1, SW3 B_2, SW4 B_3, SW5 B_4, SW6 B_5, SW7 B_6, SW8 B_7, SW9 B_8, U1 ch32v307vct6, U2 ADA4077-1xR, U3 COM-09032, U4 LM1117-3.3, U5 CH32V003, U6 CH32V003, U7 ADA4077-1xR, U8 L7805, Y1 Crystal

Commit message: + proj
Parts:
- removed Q4, Q6: Q_NMOS_GDS, Package_TO_SOT_SMD:SOT-223
- added C27: 1uF, Capacitor_SMD:C_0603_1608Metric, F.Cu at (68.1, 108.7)
- added C28: 1uF, Capacitor_SMD:C_0603_1608Metric, F.Cu at (67.7, 111.1)
- added C29: 1 nF, Capacitor_SMD:C_0603_1608Metric, F.Cu at (66.8, 114.5)
- added C30: C_Polarized, Capacitor_THT:CP_Radial_D8.0mm_P3.80mm, B.Cu at (90.6, 67.2)
- added D3: ads8863, Package_SO:VSSOP-10_3x3mm_P0.5mm, B.Cu at (67.5, 110.2)
- added D4: 1N4001, Diode_THT:D_DO-41_SOD81_P10.16mm_Horizontal, F.Cu at (123.2, 92.1)
- added D6: 1N4001, Diode_THT:D_DO-41_SOD81_P10.16mm_Horizontal, F.Cu at (96.0, 67.5)
- added J12: Conn_02x01, Connector_PinHeader_2.54mm:PinHeader_1x02_P2.54mm_Vertical, F.Cu at (84.8, 52.2)
- added J2: Conn_01x03_Male, Connector_PinHeader_2.54mm:PinHeader_1x03_P2.54mm_Vertical, F.Cu at (52.5, 108.7)
- added R27: 10k, Resistor_SMD:R_0603_1608Metric, F.Cu at (90.5, 61.2)
- added R28: 10k, Resistor_SMD:R_0603_1608Metric, F.Cu at (93.8, 61.2)
- added R29: 100, Resistor_SMD:R_0603_1608Metric, F.Cu at (105.2, 75.9)
- J7: footprint Connector_PinSocket_2.00mm:PinSocket_1x04_P2.00mm_Vertical -> Connector_PinSocket_2.54mm:PinSocket_1x04_P2.54mm_Vertical
- Q3: value Q_NMOS_GDS -> BC547; footprint Package_TO_SOT_SMD:SOT-223 -> Package_TO_SOT_THT:TO-92_Inline; moved to F.Cu
- R15: value 1,2k -> 1k
- moved Q3 28.0 mm to (108.0, 76.0), turned to -90 degrees
- moved C16 20.9 mm to (94.8, 81.9)
- moved D5 8.05 mm to (125.6, 58.8)
- moved Q8 8.00 mm to (125.8, 66.5)
- moved Q9 6.72 mm to (116.8, 66.5)
- moved R15 4.26 mm to (101.2, 76.6)
- moved C15 1.72 mm to (134.7, 98.8)
- moved C10 1.50 mm to (80.7, 51.9)
- moved C18 1.44 mm to (133.8, 96.3)
- moved J7 0.83 mm to (131.2, 51.8)
Connections:
- C11 pad 1: /VDD -> /+5
- C16 pad 2: /B+ -> /+5
- C20 pad 1: /ADC_+5 -> Net-(C20-Pad1)
- C21 pad 2: /ADC_+5 -> Net-(C20-Pad1)
- C8 pad 2: /+5 -> Net-(C8-Pad2)
- C9 pad 2: /+5 -> Net-(C8-Pad2)
- F1 pad 1: /V_BUS -> /+5
- J10 pad 3: /V_BUS -> /+5
- J11 pad 1: /V_BUS -> /+5
- J3 pad A4: /+5 -> Net-(C8-Pad2)
- J3 pad A9: /+5 -> Net-(C8-Pad2)
- J3 pad B4: /+5 -> Net-(C8-Pad2)
- J3 pad B9: /+5 -> Net-(C8-Pad2)
- J4 pad 22: Earth -> /SDCS
- J5 pad A4: /V_BUS -> /+5
- J5 pad A9: /V_BUS -> /+5
- J5 pad B4: /V_BUS -> /+5
- J5 pad B9: /V_BUS -> /+5
- J8 pad 3: /VDD -> /+5
- L2 pad 2: Net-(L2-Pad2) -> Net-(D4-Pad2)
- L3 pad 2: Net-(L3-Pad2) -> Net-(D6-Pad2)
- Q2 pad 2: Net-(L2-Pad2) -> Net-(D4-Pad2)
- Q2 pad 4: Net-(L2-Pad2) -> (no net)
- Q3 pad 1: /PWM_BOOST_N -> Net-(Q5-Pad1)
- Q3 pad 2: Net-(L2-Pad2) -> Net-(Q3-Pad2)
- Q3 pad 3: Net-(C15-Pad1) -> Earth
- Q5 pad 2: Net-(L3-Pad2) -> Net-(D6-Pad2)
- Q5 pad 4: Net-(L3-Pad2) -> (no net)
- Q7 pad 4: Net-(L1-Pad2) -> (no net)
- R15 pad 1: /V_BUS -> Net-(Q3-Pad2)
- R15 pad 2: Net-(R15-Pad2) -> Net-(U6-Pad17)
- R24 pad 2: /V_BUS -> /+5
- R26 pad 1: /VDD -> unconnected-(R26-Pad1)
- U1 pad 26: unconnected-(U1-Pad26) -> /ADC_CONVST
- U1 pad 30: unconnected-(U1-Pad30) -> /ADC_CLK
- U1 pad 31: unconnected-(U1-Pad31) -> /ADC_MISO
- U1 pad 32: unconnected-(U1-Pad32) -> /ADC_MOSI
- U1 pad 34: unconnected-(U1-Pad34) -> /ADC_START
- U1 pad 70: /USB_D- -> unconnected-(U1-Pad70)
- U1 pad 71: /USB_D+ -> unconnected-(U1-Pad71)
- U1 pad 92: unconnected-(U1-Pad92) -> /USB_D-
- U1 pad 93: unconnected-(U1-Pad93) -> /USB_D+
- U2 pad 7: /+5 -> Net-(C8-Pad2)
- U4 pad 3: /+5 -> Net-(C8-Pad2)
- U4 pad VDD: /VDD -> (no net)
- U5 pad 14: unconnected-(U5-Pad14) -> /B+
- U5 pad 9: /VDD -> /+5
- U6 pad 17: Net-(Q5-Pad1) -> Net-(U6-Pad17)
- U6 pad 19: Net-(Q6-Pad1) -> unconnected-(U6-Pad19)
- U6 pad 8: Net-(R15-Pad2) -> unconnected-(U6-Pad8)
- U6 pad 9: Net-(Q4-Pad3) -> /+5
- U8 pad 1: /ADC_+5 -> Net-(C20-Pad1)
Routing:
- net /+5: track 134.9 -> 266.2 mm, vias 6 -> 9
- net /V_BUS: track 122.1 -> 0.00 mm, vias 4 -> 0
- net /VDD: track 292.4 -> 227.8 mm, vias 18 -> 17
- net Net-(C8-Pad2): track 0.00 -> 60.3 mm, vias 0 -> 5
- net Net-(L2-Pad2): track 39.9 -> 0.00 mm
- net Net-(L3-Pad2): track 39.4 -> 0.00 mm
- net /ADC_START: track 0.00 -> 39.0 mm, vias 0 -> 3
- net Earth: track 103.6 -> 141.3 mm, vias 14 -> 34
- net /ADC_CONVST: track 0.00 -> 32.5 mm, vias 0 -> 3
- net /ADC_CLK: track 0.00 -> 31.6 mm, vias 0 -> 1
- net /ADC_MISO: track 0.00 -> 31.6 mm, vias 0 -> 1
- net Net-(D4-Pad2): track 0.00 -> 31.5 mm
- net /ADC_MOSI: track 0.00 -> 31.2 mm, vias 0 -> 1
- net /PWM_BOOST_N: track 30.7 -> 0.00 mm, vias 5 -> 0
- net Net-(D6-Pad2): track 0.00 -> 28.8 mm
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Other:
- outline, holes or cut-outs redrawn
