File: linux/tutorials/modules/usb_display/schematic/usb_display/usb_display.kicad_sch (KiCad schematic)
At the start: 105 parts, among them J1 Conn_01x04_Male, J10 Conn_01x03_Male, J11 Conn_02x01, J3 USB_C_Receptacle_USB2.0, J4 Conn_02x17_Odd_Even, J5 USB_C_Receptacle_USB2.0, J6 Conn_02x01, J7 Screw_Terminal_01x04, J8 Conn_01x03_Male, J9 Conn_02x01, Q1 BD250, Q2 Q_NMOS_GDS, Q3 Q_NMOS_GDS, Q4 Q_NMOS_GDS, Q5 Q_NMOS_GDS, Q6 Q_NMOS_GDS, Q7 Q_NMOS_GDS, Q8 Q_NMOS_GDS, Q9 Q_NMOS_GDS, SW1 B_0, SW10 B_9, SW11 B_10, SW12 B_11, SW13 B_12, SW14 B_13, SW15 B_14, SW16 B_15, SW17 SW_Push_Rst, SW18 B_ENTER, SW2 B_1, SW3 B_2, SW4 B_3, SW5 B_4, SW6 B_5, SW7 B_6, SW8 B_7, SW9 B_8, U1 ch32v307vct6, U2 ADA4077-1xR, U3 COM-09032, U4 LM1117-3.3, U5 CH32V003, U6 CH32V003, U7 ADA4077-1xR, U8 L7805, Y1 Crystal

Commit message: + proj
Parts:
- removed Q3, Q4, Q6: Q_NMOS_GDS, Package_TO_SOT_SMD:SOT-223, symbol Device:Q_NMOS_GDS
- added C27, C28: 1uF, Capacitor_SMD:C_0603_1608Metric, symbol Device:C
- added C29: 1 nF, Capacitor_SMD:C_0603_1608Metric, symbol Device:C
- added C30: C_Polarized, Capacitor_THT:CP_Radial_D8.0mm_P3.80mm, symbol Device:C_Polarized
- added D3: ads8863, Package_SO:VSSOP-10_3x3mm_P0.5mm, symbol New_Library:ads8863
- added D4, D6: 1N4001, Diode_THT:D_DO-41_SOD81_P10.16mm_Horizontal, symbol Diode:1N4001
- added J12: Conn_02x01, Connector_PinHeader_2.54mm:PinHeader_1x02_P2.54mm_Vertical, symbol Connector_Generic:Conn_02x01
- added J2: Conn_01x03_Male, Connector_PinHeader_2.54mm:PinHeader_1x03_P2.54mm_Vertical, symbol Connector:Conn_01x03_Male
- added Q3: BC547, Package_TO_SOT_THT:TO-92_Inline, symbol Transistor_BJT:BC547
- added R27, R28: 10k, Resistor_SMD:R_0603_1608Metric, symbol Device:R
- added R29: 100, Resistor_SMD:R_0603_1608Metric, symbol Device:R_Small
- J7: footprint Connector_PinSocket_2.00mm:PinSocket_1x04_P2.00mm_Vertical -> Connector_PinSocket_2.54mm:PinSocket_1x04_P2.54mm_Vertical
- R15: value 1,2k -> 1k
Connections:
- net +5: now also C11.1, C16.2, F1.1, J10.3 (Pin_3), J11.1 (Pin_1), J5.A4 (VBUS), J5.A9 (VBUS), J5.B4 (VBUS), J5.B9 (VBUS), J8.3 (Pin_3), R24.2, U5.9 (VDD), U6.9 (VDD), C30.1, J12.2 (Pin_2), R29.1; no longer C8.2, C9.2, J3.A4 (VBUS), J3.A9 (VBUS), J3.B4 (VBUS), J3.B9 (VBUS), U2.7 (V+), U4.3 (VI)
- net ADC_+5: now also R27.1, R28.1; no longer C20.1, C21.2, U8.1 (IN)
- net B+: now also U5.14 (PC4); no longer C16.2
- net Earth: now also C27.1, C28.1, C29.1, C30.2, D3.4 (AINN), D3.5 (GND), J2.3 (Pin_3), Q3.3 (E), R28.2
- net USB_D+: now also U1.93 (PB7); no longer U1.71 (PA12)
- net USB_D-: now also U1.92 (PB6); no longer U1.70 (PA11)
- net VDD: now also C27.2, D3.10 (DVDD); no longer C11.1, J8.3 (Pin_3), R26.1, U5.9 (VDD)
- net at C15.1, C17.2, C18.2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: now also D4.1 (K)
- net at L3.2, Q5.2 (D): now also D6.2 (A)
- net at Q5.1 (G): now also Q3.1 (C), R29.2; no longer U6.17 (PC7)
- net at R15.2: now also U6.17 (PC7); no longer U6.8 (PD0)
- net ADC_CONVST: now reaches U1.26 (PA3)
- net ADC_CONVST: now also D3.6 (CONVST)
- net ADC_CLK: now reaches U1.30 (PA5)
- net ADC_CLK: now also D3.8 (SCLK)
- net ADC_MISO: now reaches U1.31 (PA6)
- net ADC_MISO: now also D3.7 (DOUT)
- net ADC_MOSI: now reaches U1.32 (PA7)
- net ADC_MOSI: now also D3.9 (DIN)
- net ADC_START: now reaches U1.34 (PC5)
- net ADC_START: now also J2.1 (Pin_1)
- net at L2.2, Q2.2 (D): now also D4.2 (A)
- removed net V_BUS: F1.1, J10.3 (Pin_3), J11.1 (Pin_1), J5.A4 (VBUS), J5.A9 (VBUS), J5.B4 (VBUS), J5.B9 (VBUS), R15.1, R24.2
- new net: C29.2, D3.3 (AINP), J2.2 (Pin_2)
- new net: C20.1, C21.2, D6.1 (K), R27.2, U8.1 (IN)
- new net: C8.2, C9.2, J12.1 (Pin_1), J3.A4 (VBUS), J3.A9 (VBUS), J3.B4 (VBUS), J3.B9 (VBUS), U2.7 (V+), U4.3 (VI)
- new net: C28.2, D3.1 (REF), D3.2 (AVDD)
- new net: Q3.2 (B), R15.1
Other:
- moved on the sheet: C10, Q5, R26, U4
